File: BlueESC/Logic.sch (EAGLE design)
At the start: 36 parts, among them U1 ATMEGA168, U2 V_REG_LDOSMD, Y1 RESONATORSMD

Commit message: Updated PWM pull down to 470K to avoid avoid beating out the internal pull-ups used in ArduinoUSBLinker.
Parts:
- R16: value 10K -> 4.7K
- R18: value 10K -> 470K
Changed lines of the file:
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@@
 <?xml version="1.0" encoding="utf-8"?>
 <!DOCTYPE eagle SYSTEM "eagle.dtd">
-<eagle version="7.1.0">
+<eagle version="7.4.0">
 <drawing>
 <settings>
@@
 <part name="Y1" library="SparkFun" deviceset="RESONATOR" device="SMD"/>
 <part name="R15" library="SparkFun" deviceset="RESISTOR" device="0603-RES" value="1K"/>
-<part name="R16" library="SparkFun" deviceset="RESISTOR" device="0603-RES" value="10K"/>
+<part name="R16" library="SparkFun" deviceset="RESISTOR" device="0603-RES" value="4.7K"/>
 <part name="GND7" library="SparkFun" deviceset="GND" device=""/>
 <part name="C7" library="SparkFun-Capacitors" deviceset="CAP" device="0603-CAP" value="0.1uF"/>
@@
 <part name="LED1" library="BR-Eagle-Library" deviceset="LED" device="3X2-RA" value="BLUE"/>
 <part name="LED2" library="BR-Eagle-Library" deviceset="LED" device="3X2-RA" value="RED"/>
-<part name="R18" library="SparkFun" deviceset="RESISTOR" device="0603-RES" value="10K"/>
+<part name="R18" library="SparkFun" deviceset="RESISTOR" device="0603-RES" value="470K"/>
 <part name="GND6" library="SparkFun" deviceset="GND" device=""/>
 </parts>
